File: CC_M7/RF Telemetry.kicad_sch (KiCad schematic)
At the start: 30 parts, among them J9 SMA_CONNECTOR, U6 nRF52820-QDxx, U7 NRF21540-QDAA-R7, Y2 32MHz

Commit message: Scehmatic completed.
Parts:
- C58: footprint (none) -> Capacitor_SMD:C_0402_1005Metric
Changed lines of the file:
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@@
 			)
 		)
-		(property "Footprint" ""
+		(property "Footprint" "Capacitor_SMD:C_0402_1005Metric"
 			(at 71.12 182.88 0)
 			(effects

Commit message: last control
Connections:
- net J2_36 is gone; now on net J2_32: JP6.2 (B)
- net J2_32: no longer JP5.2 (B)
- net NRF_SWCLK: now also JP7.1 (A); no longer JP6.1 (A)
- net NRF_SWDIO: now also JP6.1 (A); no longer JP7.1 (A)
- net J2_38 renamed J2_34
- new net J2_31: JP5.2 (B)
Other:
- note added: "SWDEBUG"
- note removed: "SWO"
- moved on the sheet: JP5, JP6, JP7, JP8
Changed lines of the file:
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@@
 		)
 	)
-	(text "SWO"
+	(text "SWDEBUG"
 		(exclude_from_sim no)
-		(at 195.58 81.28 0)
+		(at 193.04 78.74 0)
 		(effects
 			(font
@@
 	(global_label "NRF_SWCLK"
 		(shape input)
-		(at 170.18 66.04 180)
+		(at 170.18 68.58 180)
 		(fields_autoplaced yes)
 		(effects
@@
 		)
 		(property "Intersheetrefs" "${INTERSHEET_REFS}"
-			(at 156.3091 66.04 0)
+			(at 156.3091 68.58 0)
 			(effects
 				(font
@@
 	(global_label "NRF_NRST"
 		(shape input)
-		(at 170.18 76.2 180)
+		(at 170.18 73.66 180)
 		(fields_autoplaced yes)
 		(effects
@@
 		)
 		(property "Intersheetrefs" "${INTERSHEET_REFS}"
-			(at 157.7605 76.2 0)
+			(at 157.7605 73.66 0)
 			(effects
 				(font
@@
 		)
 	)
-	(global_label "J2_38"
-		(shape input)
-		(at 180.34 71.12 0)
-		(fields_autoplaced yes)
-		(effects
-			(font
-				(size 1.27 1.27)
-			)
-			(justify left)
-		)
-		(property "Intersheetrefs" "${INTERSHEET_REFS}"
-			(at 188.8889 71.12 0)
-			(effects
-				(font
-					(size 1.27 1.27)
-				)
-				(justify left)
-				(hide yes)
-			)
-		)
-	)
 	(global_label "NRF_ANT"
 		(shape bidirectional)
@@
 		)
 	)
+	(global_label "J2_32"
+		(shape input)
+		(at 180.34 63.5 0)
+		(fields_autoplaced yes)
+		(effects
+			(font
+				(size 1.27 1.27)
+			)
+			(justify left)
+		)
+		(property "Intersheetrefs" "${INTERSHEET_REFS}"
+			(at 188.8889 63.5 0)
+			(effects
+				(font
+					(size 1.27 1.27)
+				)
+				(justify left)
+				(hide yes)
+			)
+		)
+	)
+	(global_label "J2_31"
+		(shape input)
+		(at 180.34 58.42 0)
+		(fields_autoplaced yes)
+		(effects
+			(font
+				(size 1.27 1.27)
+			)
+			(justify left)
+		)
+		(property "Intersheetrefs" "${INTERSHEET_REFS}"
+			(at 188.8889 58.42 0)
+			(effects
+				(font
+					(size 1.27 1.27)
+				)
+				(justify left)
+				(hide yes)
+			)
+		)
+	)
 	(global_label "NRF_XC1"
 		(shape input)
@@
 		)
 	)
+	(global_label "J2_34"
+		(shape input)
+		(at 180.34 68.58 0)
+		(fields_autoplaced yes)
+		(effects
+			(font
+				(size 1.27 1.27)
+			)
+			(justify left)
+		)
+		(property "Intersheetrefs" "${INTERSHEET_REFS}"
+			(at 188.8889 68.58 0)
+			(effects
+				(font
+					(size 1.27 1.27)
+				)
+				(justify left)
+				(hide yes)
+			)
+		)
+	)
 	(global_label "3V3_RF"
 		(shape input)
@@
 	(global_label "NRF_SWDIO"
 		(shape input)
-		(at 170.18 71.12 180)
+		(at 170.18 63.5 180)
 		(fields_autoplaced yes)
 		(effects
@@
 		)
 		(property "Intersheetrefs" "${INTERSHEET_REFS}"
-			(at 156.6719 71.12 0)
+			(at 156.6719 63.5 0)
 			(effects
 				(font
@@
 	(global_label "3V3_RF"
 		(shape input)
-		(at 170.18 60.96 180)
+		(at 170.18 58.42 180)
 		(fields_autoplaced yes)
 		(effects
@@
 		)
 		(property "Intersheetrefs" "${INTERSHEET_REFS}"
-			(at 160.361 60.96 0)
+			(at 160.361 58.42 0)
 			(effects
 				(font
@@
 	(global_label "J2_40"
 		(shape input)
-		(at 180.34 76.2 0)
+		(at 180.34 73.66 0)
 		(fields_autoplaced yes)
 		(effects
@@
 		)
 		(property "Intersheetrefs" "${INTERSHEET_REFS}"
-			(at 188.8889 76.2 0)
+			(at 188.8889 73.66 0)
 			(effects
 				(font
@@
 		)
 	)
-	(global_label "J2_32"
-		(shape input)
-		(at 180.34 60.96 0)
-		(fields_autoplaced yes)
-		(effects
-			(font
-				(size 1.27 1.27)
-			)
-			(justify left)
-		)
-		(property "Intersheetrefs" "${INTERSHEET_REFS}"
-			(at 188.8889 60.96 0)
-			(effects
-				(font
-					(size 1.27 1.27)
-				)
-				(justify left)
-				(hide yes)
-			)
-		)
-	)
 	(global_label "3V3_RF"
 		(shape input)
@@
 		)
 	)
-	(global_label "J2_36"
-		(shape input)
-		(at 180.34 66.04 0)
-		(fields_autoplaced yes)
-		(effects
-			(font
-				(size 1.27 1.27)
-			)
-			(justify left)
-		)
-		(property "Intersheetrefs" "${INTERSHEET_REFS}"
-			(at 188.8889 66.04 0)
-			(effects
-				(font
-					(size 1.27 1.27)
-				)
-				(justify left)
-				(hide yes)
-			)
-		)
-	)
 	(global_label "NRF_XC2"
 		(shape input)
@@
 	(symbol
 		(lib_id "Jumper:Jumper_2_Bridged")
-		(at 175.26 66.04 0)
+		(at 175.26 63.5 0)
 		(unit 1)
 		(exclude_from_sim yes)
@@
 		(dnp no)
 		(property "Reference" "JP6"
-			(at 175.26 63.5 0)
+			(at 175.26 60.96 0)
 			(effects
 				(font
@@
 		)
 		(property "Value" "SWDIO"
-			(at 175.26 63.5 0)
+			(at 175.26 60.96 0)
 			(effects
 				(font
@@
 		)
 		(property "Footprint" "jmpertest:jmpertest"
-			(at 175.26 66.04 0)
+			(at 175.26 63.5 0)
 			(effects
 				(font
@@
 		)
 		(property "Datasheet" "~"
-			(at 175.26 66.04 0)
+			(at 175.26 63.5 0)
 			(effects
 				(font
@@
 		)
 		(property "Description" "Jumper, 2-pole, closed/bridged"
-			(at 175.26 66.04 0)
+			(at 175.26 63.5 0)
 			(effects
 				(font
@@
 	(symbol
 		(lib_id "Jumper:Jumper_2_Bridged")
-		(at 175.26 71.12 0)
+		(at 175.26 68.58 0)
 		(unit 1)
 		(exclude_from_sim yes)
@@
 		(dnp no)
 		(property "Reference" "JP7"
-			(at 175.26 68.58 0)
+			(at 175.26 66.04 0)
 			(effects
 				(font
@@
 		)
 		(property "Value" "SWDIO"
-			(at 175.26 68.58 0)
+			(at 175.26 66.04 0)
 			(effects
 				(font
@@
 		)
 		(property "Footprint" "jmpertest:jmpertest"
-			(at 175.26 71.12 0)
+			(at 175.26 68.58 0)
 			(effects
 				(font
@@
 		)
 		(property "Datasheet" "~"
-			(at 175.26 71.12 0)
+			(at 175.26 68.58 0)
 			(effects
 				(font
@@
 		)
 		(property "Description" "Jumper, 2-pole, closed/bridged"
-			(at 175.26 71.12 0)
+			(at 175.26 68.58 0)
 			(effects
 				(font
@@
 	(symbol
 		(lib_id "Jumper:Jumper_2_Bridged")
-		(at 175.26 60.96 0)
+		(at 175.26 58.42 0)
 		(unit 1)
 		(exclude_from_sim yes)
@@
 		(dnp no)
 		(property "Reference" "JP5"
-			(at 175.26 58.42 0)
+			(at 175.26 55.88 0)
 			(effects
 				(font
@@
 		)
 		(property "Value" "SWDIO"
-			(at 175.26 58.42 0)
+			(at 175.26 55.88 0)
 			(effects
 				(font
@@
 		)
 		(property "Footprint" "jmpertest:jmpertest"
-			(at 175.26 60.96 0)
+			(at 175.26 58.42 0)
 			(effects
 				(font
@@
 		)
 		(property "Datasheet" "~"
-			(at 175.26 60.96 0)
+			(at 175.26 58.42 0)
 			(effects
 				(font
@@
 		)
 		(property "Description" "Jumper, 2-pole, closed/bridged"
-			(at 175.26 60.96 0)
+			(at 175.26 58.42 0)
 			(effects
 				(font
@@
 	(symbol
 		(lib_id "Jumper:Jumper_2_Bridged")
-		(at 175.26 76.2 0)
+		(at 175.26 73.66 0)
 		(unit 1)
 		(exclude_from_sim yes)
@@
 		(dnp no)
 		(property "Reference" "JP8"
-			(at 175.26 73.66 0)
+			(at 175.26 71.12 0)
 			(effects
 				(font
@@
 		)
 		(property "Value" "SWDIO"
-			(at 175.26 73.66 0)
+			(at 175.26 71.12 0)
 			(effects
 				(font
@@
 		)
 		(property "Footprint" "jmpertest:jmpertest"
-			(at 175.26 76.2 0)
+			(at 175.26 73.66 0)
 			(effects
 				(font
@@
 		)
 		(property "Datasheet" "~"
-			(at 175.26 76.2 0)
+			(at 175.26 73.66 0)
 			(effects
 				(font
@@
 		)
 		(property "Description" "Jumper, 2-pole, closed/bridged"
-			(at 175.26 76.2 0)
+			(at 175.26 73.66 0)
 			(effects
 				(font

Commit message: ready for routing
Parts:
- removed JP5: SWDIO, jmpertest:jmpertest, symbol Jumper:Jumper_2_Bridged
- added JP10, JP9: SWDIO, Jumper:SolderJumper-2_P1.3mm_Open_TrianglePad1.0x1.5mm, symbol Jumper:Jumper_2_Bridged
- C28, C29, C31, C32, C33, C37, C38, C41, C42, C44: footprint Capacitor_SMD:C_0201_0603Metric -> Capacitor_SMD:C_0402_1005Metric
- JP6, JP7, JP8: footprint jmpertest:jmpertest -> Jumper:SolderJumper-2_P1.3mm_Open_TrianglePad1.0x1.5mm
Connections:
- net 3V3_RF: now also JP6.2 (B)
- net J2_31: now also JP6.1 (A)
- net J2_32: now also JP7.1 (A); no longer JP6.2 (B)
- net J2_34: now also JP8.1 (A); no longer JP7.2 (B)
- net J2_40: now also JP10.1 (A); no longer JP8.2 (B)
- net NRF_NRST: now also JP10.2 (B); no longer JP8.1 (A)
- net NRF_SWCLK: now also JP8.2 (B); no longer JP7.1 (A)
- net NRF_SWDIO: now also JP7.2 (B); no longer JP6.1 (A)
- no-connect marks 6 -> 8
Other:
- note added: "NO USB: D+ : NC D- : NC DECUSB : NC VBUS : GND"
- note removed: "Kontrol Yapılacak!!!!!"

Commit message: CCM7A BIG ROUTING PROGRESS
Parts:
- L6, L7: footprint Inductor_SMD:L_0201_0603Metric -> Inductor_SMD:L_0402_1005Metric
Changed lines of the file:
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@@
 			)
 		)
-		(property "Footprint" "Inductor_SMD:L_0201_0603Metric"
+		(property "Footprint" "Inductor_SMD:L_0402_1005Metric"
 			(at 132.08 177.8 0)
 			(effects
@@
 			)
 		)
-		(property "Footprint" "Inductor_SMD:L_0201_0603Metric"
+		(property "Footprint" "Inductor_SMD:L_0402_1005Metric"
 			(at 121.92 177.8 0)
 			(effects

Commit message: Debugging routes added. / Debug footprint updated.
Connections:
- net J2_36: now reaches JP9.1 (A)
- no-connect marks 8 -> 7
Changed lines of the file:
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@@
-	)
-	(no_connect
-		(at 165.1 73.66)
 	)
 	(no_connect
@@
 			(effects
 				(font
+					(size 1.27 1.27)
+				)
+				(justify right)
+				(hide yes)
+			)
+		)
+	)
+	(global_label "J2_36"
+		(shape input)
+		(at 165.1 73.66 180)
+		(fields_autoplaced yes)
+		(effects
+			(font
+				(size 1.27 1.27)
+			)
+			(justify right)
+		)
+		(property "Intersheetrefs" "${INTERSHEET_REFS}"
+			(at 156.5511 73.66 0)
+			(effects
+				(font

Commit message: BOM finished.
Parts:
- C32, C44: value 16pF -> 8pF
- D5, D6: footprint LED_SMD:LED_0402_1005Metric -> LED_SMD:LED_0805_2012Metric
Changed lines of the file:
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@@
 			)
 		)
-		(property "Footprint" "LED_SMD:LED_0402_1005Metric"
+		(property "Footprint" "LED_SMD:LED_0805_2012Metric"
 			(at 168.91 132.08 0)
 			(effects
@@
 			)
 		)
-		(property "Footprint" "LED_SMD:LED_0402_1005Metric"
+		(property "Footprint" "LED_SMD:LED_0805_2012Metric"
 			(at 168.91 124.46 0)
 			(effects
@@
 			)
 		)
-		(property "Value" "16pF"
+		(property "Value" "8pF"
 			(at 185.42 100.3235 0)
 			(effects
@@
 			)
 		)
-		(property "Value" "16pF"
+		(property "Value" "8pF"
 			(at 154.94 100.33 0)
 			(effects
