File: CC_M7/RF Telemetry.kicad_sch (KiCad schematic)
At the start: 31 parts, among them J9 SMA_CONNECTOR, U6 nRF52820-QDxx, U7 NRF21540-QDAA-R7, Y2 32MHz

Commit message: last check
Parts:
- C28, C29, C58: footprint Capacitor_SMD:C_0402_1005Metric -> Capacitor_SMD:C_0201_0603Metric
- L6, L7: footprint Inductor_SMD:L_0402_1005Metric -> Inductor_SMD:L_0201_0603Metric
Changed lines of the file:
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@@
 			)
 		)
-		(property "Footprint" "Inductor_SMD:L_0402_1005Metric"
+		(property "Footprint" "Inductor_SMD:L_0201_0603Metric"
 			(at 132.08 177.8 0)
 			(effects
@@
 			)
 		)
-		(property "Footprint" "Capacitor_SMD:C_0402_1005Metric"
+		(property "Footprint" "Capacitor_SMD:C_0201_0603Metric"
 			(at 142.24 182.88 0)
 			(effects
@@
 			)
 		)
-		(property "Footprint" "Capacitor_SMD:C_0402_1005Metric"
+		(property "Footprint" "Capacitor_SMD:C_0201_0603Metric"
 			(at 71.12 182.88 0)
 			(effects
@@
 			)
 		)
-		(property "Footprint" "Capacitor_SMD:C_0402_1005Metric"
+		(property "Footprint" "Capacitor_SMD:C_0201_0603Metric"
 			(at 127 182.88 0)
 			(effects
@@
 			)
 		)
-		(property "Footprint" "Inductor_SMD:L_0402_1005Metric"
+		(property "Footprint" "Inductor_SMD:L_0201_0603Metric"
 			(at 121.92 177.8 0)
 			(effects

Commit message: ...
Parts:
- added C61: 1pF, Capacitor_SMD:C_0201_0603Metric, symbol Device:C_Small
- added C62: 1.2pF, Capacitor_SMD:C_0201_0603Metric, symbol Device:C_Small
- added L2: 4.7nH, Inductor_SMD:L_0201_0603Metric, symbol Device:L_Small
- added L3: 2.2nH, Inductor_SMD:L_0201_0603Metric, symbol Device:L_Small
Connections:
- net GND: now also C61.2, C62.2
- net NRF_ANT: now also L3.1; no longer U6.24 (ANT)
- new net: C62.1, L2.1, L3.2
- new net: C61.1, L2.2, U6.24 (ANT)
Other:
- moved on the sheet: U6

Commit message: pdf added
Parts:
- C31: footprint Capacitor_SMD:C_0402_1005Metric -> Capacitor_SMD:C_0201_0603Metric
Changed lines of the file:
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@@
 			)
 		)
-		(property "Footprint" "Capacitor_SMD:C_0402_1005Metric"
+		(property "Footprint" "Capacitor_SMD:C_0201_0603Metric"
 			(at 134.62 38.1 0)
 			(effects
