File: CC_M7/CC_M7.kicad_sch (KiCad schematic)
At the start: 6 parts

Commit message: ready for routing
Other:
- note added: "STM32H743VGT6 Pins Connections Voltage Read Filters Stm32h743 Requirments"
- note removed: "STM32H743VIT6 Pins Connections Voltage Read Filters Stm32h743 Requirments"
Changed lines of the file:
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@@
 		)
 	)
-	(text "STM32H743VIT6 Pins Connections\nVoltage Read\nFilters\nStm32h743 Requirments"
+	(text "STM32H743VGT6 Pins Connections\nVoltage Read\nFilters\nStm32h743 Requirments"
 		(exclude_from_sim no)
 		(at 29.972 25.4 0)
