File: CC_M7/Sensors.kicad_sch (KiCad schematic)
At the start: 14 parts, among them U11 BMP581, U2 24AA64T-I/OT, U3 BMI088, U4 ICP-20100, U5 BMM150

Commit message: Scehmatic completed.
Parts:
- removed C26, C27: 100nF, Capacitor_SMD:C_0402_1005Metric, symbol Device:C_Small
- removed U5: BMM150, Package_CSP:WLCSP-12_1.56x1.56mm_P0.4mm, symbol Sensor_Magnetic:BMM150
- added C52, C56, C57: 100nF, Capacitor_SMD:C_0402_1005Metric, symbol Device:C_Small
- added U13: ICM-20948, Sensor_Motion:InvenSense_QFN-24_3x3mm_P0.4mm, symbol Sensor_Motion:ICM-20948
- added U5: TXB0104RUT, Package_DFN_QFN:Texas_R-PUQFN-N12, symbol Logic_LevelTranslator:TXB0104RUT
- R11: value 1k -> 10k
Connections:
- net I2C1_IRQ3 is gone; now on net I2C1_IRQ2: U4.7 (INT)
- net +3.3V: now also U5.11 (VCCB)
- net GND: now also R11.1, U11.5 (SDO), C52.2, C56.2, C57.2, U13.11 (FSYNC), U13.18 (GND), U13.20 (GND), U5.6 (GND)
- net I2C1_IRQ2: no longer R11.2
- net SPI1_MISO: now also U5.8 (B3)
- net SPI1_MOSI: now also U5.9 (B2)
- net SPI1_SCK: now also U5.7 (B4)
- new net: C57.1, U13.10 (REGOUT)
- new net +1V8: C52.1, C56.1, R11.2, U13.13 (VDD), U13.8 (VDDIO), U5.1 (VCCA), U5.12 (OE)
- new net SPI1_CS3: U5.10 (B1)
- new net SPI1_CS3_1V8: U13.22 (~{CS}), U5.2 (A1)
- new net SPI1_MISO_1V8: U13.9 (SDO/AD0), U5.4 (A3)
- new net SPI1_MOSI_1V8: U13.24 (SDA/SDI), U5.3 (A2)
- new net SPI1_SCK_1V8: U13.23 (SCL/SCLK), U5.5 (A4)
- no-connect marks 7 -> 8
Other:
- note added: "24AA64"
- note added: "ICM20948"
- note added: "ICP20100"
- note removed: "BMM150"
- note removed: "EEPROM"
- note removed: "ICP-20100"
- note removed: "ICP-20948"
- note removed: "The capacitors will be close to the VDD and VDDIO pins. I²C address bit 0: SDO --> GND: '0'; VDDIO: '1' I²C address bit 1: CSB --> GND: '0'; VDDIO: '1'"
- moved on the sheet: C22, C23, C24, C25, C54, C55, U11, U2, U3, U4

Commit message: CCM7A Routing in progress.
Connections:
- net SPI1_CS3: now also U5.7 (B4); no longer U5.10 (B1)
- net SPI1_CS3_1V8: now also U5.5 (A4); no longer U5.2 (A1)
- net SPI1_MISO: now also U5.9 (B2); no longer U5.8 (B3)
- net SPI1_MISO_1V8: now also U5.3 (A2); no longer U5.4 (A3)
- net SPI1_MOSI: now also U5.8 (B3); no longer U5.9 (B2)
- net SPI1_MOSI_1V8: now also U5.4 (A3); no longer U5.3 (A2)
- net SPI1_SCK: now also U5.10 (B1); no longer U5.7 (B4)
- net SPI1_SCK_1V8: now also U5.2 (A1); no longer U5.5 (A4)
Changed lines of the file:
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@@
 	(global_label "SPI1_MISO"
 		(shape input)
-		(at 167.64 208.28 0)
+		(at 167.64 203.2 0)
 		(fields_autoplaced yes)
 		(effects
@@
 		)
 		(property "Intersheetrefs" "${INTERSHEET_REFS}"
-			(at 180.4828 208.28 0)
+			(at 180.4828 203.2 0)
 			(effects
 				(font
@@
 	(global_label "SPI1_MOSI"
 		(shape input)
-		(at 167.64 203.2 0)
+		(at 167.64 208.28 0)
 		(fields_autoplaced yes)
 		(effects
@@
 		)
 		(property "Intersheetrefs" "${INTERSHEET_REFS}"
-			(at 180.4828 203.2 0)
+			(at 180.4828 208.28 0)
 			(effects
 				(font
@@
 	(global_label "SPI1_MOSI_1V8"
 		(shape input)
-		(at 147.32 203.2 180)
+		(at 147.32 208.28 180)
 		(fields_autoplaced yes)
 		(effects
@@
 		)
 		(property "Intersheetrefs" "${INTERSHEET_REFS}"
-			(at 130.002 203.2 0)
+			(at 130.002 208.28 0)
 			(effects
 				(font
@@
 	(global_label "SPI1_SCK_1V8"
 		(shape input)
-		(at 147.32 213.36 180)
+		(at 147.32 198.12 180)
 		(fields_autoplaced yes)
 		(effects
@@
 		)
 		(property "Intersheetrefs" "${INTERSHEET_REFS}"
-			(at 130.8487 213.36 0)
+			(at 130.8487 198.12 0)
 			(effects
 				(font
@@
 	(global_label "SPI1_CS3"
 		(shape input)
-		(at 167.64 198.12 0)
+		(at 167.64 213.36 0)
 		(fields_autoplaced yes)
 		(effects
@@
 		)
 		(property "Intersheetrefs" "${INTERSHEET_REFS}"
-			(at 179.5756 198.12 0)
+			(at 179.5756 213.36 0)
 			(effects
 				(font
@@
 	(global_label "SPI1_CS3_1V8"
 		(shape input)
-		(at 147.32 198.12 180)
+		(at 147.32 213.36 180)
 		(fields_autoplaced yes)
 		(effects
@@
 		)
 		(property "Intersheetrefs" "${INTERSHEET_REFS}"
-			(at 130.9092 198.12 0)
+			(at 130.9092 213.36 0)
 			(effects
 				(font
@@
 	(global_label "SPI1_SCK"
 		(shape input)
-		(at 167.64 213.36 0)
+		(at 167.64 198.12 0)
 		(fields_autoplaced yes)
 		(effects
@@
 		)
 		(property "Intersheetrefs" "${INTERSHEET_REFS}"
-			(at 179.6361 213.36 0)
+			(at 179.6361 198.12 0)
 			(effects
 				(font
@@
 	(global_label "SPI1_MISO_1V8"
 		(shape input)
-		(at 147.32 208.28 180)
+		(at 147.32 203.2 180)
 		(fields_autoplaced yes)
 		(effects
@@
 		)
 		(property "Intersheetrefs" "${INTERSHEET_REFS}"
-			(at 130.002 208.28 0)
+			(at 130.002 203.2 0)
 			(effects
 				(font
@@
 		)
 		(instances
-			(project ""
+			(project "CC_M7"
 				(path "/20c3bbae-00c6-470e-8b69-dc0f665257a3/b4ae7b3b-cd15-4dc2-a519-be49b0fe3ceb"
 					(reference "U5")
@@
 		)
 		(instances
-			(project ""
+			(project "CC_M7"
 				(path "/20c3bbae-00c6-470e-8b69-dc0f665257a3/b4ae7b3b-cd15-4dc2-a519-be49b0fe3ceb"
 					(reference "U13")
@@
 		)
 		(instances
-			(project ""
+			(project "CC_M7"
 				(path "/20c3bbae-00c6-470e-8b69-dc0f665257a3/b4ae7b3b-cd15-4dc2-a519-be49b0fe3ceb"
 					(reference "#PWR0113")
@@
 		)
 		(instances
-			(project ""
+			(project "CC_M7"
 				(path "/20c3bbae-00c6-470e-8b69-dc0f665257a3/b4ae7b3b-cd15-4dc2-a519-be49b0fe3ceb"
 					(reference "#PWR0105")
@@
 		)
 		(instances
-			(project ""
+			(project "CC_M7"
 				(path "/20c3bbae-00c6-470e-8b69-dc0f665257a3/b4ae7b3b-cd15-4dc2-a519-be49b0fe3ceb"
 					(reference "#PWR037")
@@
 		)
 		(instances
-			(project ""
+			(project "CC_M7"
 				(path "/20c3bbae-00c6-470e-8b69-dc0f665257a3/b4ae7b3b-cd15-4dc2-a519-be49b0fe3ceb"
 					(reference "C52")
@@
 		)
 		(instances
-			(project ""
+			(project "CC_M7"
 				(path "/20c3bbae-00c6-470e-8b69-dc0f665257a3/b4ae7b3b-cd15-4dc2-a519-be49b0fe3ceb"
 					(reference "R11")
