File: CC_M7/Power.kicad_sch (KiCad schematic)
At the start: 32 parts, among them J13 Batt_Pins, U10 ME6211C33M5, U12 TPS79318-EP, U8 TPS562206, U9 ME6211C33M5

Commit message: BOM finished.
Parts:
- L1: value SRN6045TA-2R2Y -> 2.2uH
- U8: value TPS562206 -> TPS566242DRL
Other:
- note added: "Akım ve regülatör kontrolü yapılacak!!!!"
Changed lines of the file:
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@@
 		)
 	)
+	(text "Akım ve regülatör kontrolü yapılacak!!!!"
+		(exclude_from_sim no)
+		(at 58.42 165.1 0)
+		(effects
+			(font
+				(size 2.54 2.54)
+				(thickness 0.508)
+				(bold yes)
+			)
+		)
+	)
 	(global_label "VIN_5V"
 		(shape input)
@@
 			)
 		)
-		(property "Value" "TPS562206"
+		(property "Value" "TPS566242DRL"
 			(at 93.98 38.1 0)
 			(effects
@@
 			)
 		)
-		(property "Value" "SRN6045TA-2R2Y"
+		(property "Value" "2.2uH"
 			(at 121.92 38.1 0)
 			(effects

Commit message: Finished
Parts:
- D9: value SS210 -> B5819WS
Other:
- note removed: "B5819WS"

Commit message: pdf added
Parts:
- removed D7, D8: 1N5819WS, Diode_SMD:D_SOD-323, symbol Diode:1N5819WS
- D9: value B5819WS -> BAT60B
- R18: value 33k -> 30k
Connections:
- net +3.3V: now also C50.1, U10.5 (V_{OUT})
- net 3V3_RF: now also C45.1, U9.5 (V_{OUT})
